Commit message: FIX robot mecanum urdf file robot urdf and gazebo file changed and bugs fixed

File: robot_simulation/urdf/robot.gazebo.xacro (robot description, xacro)
@@ -1,78 +1,123 @@
 <?xml version="1.0"?>
-<robot xmlns:xacro="http://www.ros.org/wiki/xacro">
-    <gazebo reference="base_footprint">
-        <material>Gazebo/Blue</material>
-    </gazebo>
-    <!-- Mecanum wheel friction properties -->
-    <gazebo reference="wheel_front_left_link">
-        <material>Gazebo/Black</material>
-        <mu1>0.8</mu1>
-        <mu2>0.8</mu2>
-    </gazebo>
-    <gazebo reference="wheel_front_right_link">
-        <material>Gazebo/Black</material>
-        <mu1>0.8</mu1>
-        <mu2>0.8</mu2>
-    </gazebo>
-    <gazebo reference="wheel_rear_left_link">
-        <material>Gazebo/Black</material>
-        <mu1>0.8</mu1>
-        <mu2>0.8</mu2>
-    </gazebo>
-    <gazebo reference="wheel_rear_right_link">
-        <material>Gazebo/Black</material>
-        <mu1>0.8</mu1>
-        <mu2>0.8</mu2>
-    </gazebo>
-    <!-- Joint State Publisher - publishes all joint states -->
-    <gazebo>
-        <plugin filename="ignition-gazebo-joint-state-publisher-system"
-                name="ignition::gazebo::systems::JointStatePublisher">
-        </plugin>
-    </gazebo>
-    <gazebo>
-  <plugin filename="libignition-gazebo6-mecanum-drive-system"
-    name="ignition::gazebo::systems::MecanumDrive">
-        <front_left_joint>wheel_front_left_joint</front_left_joint>
-        <front_right_joint>wheel_front_right_joint</front_right_joint>
-        <back_left_joint>wheel_rear_left_joint</back_left_joint>
-        <back_right_joint>wheel_rear_right_joint</back_right_joint>
-        <wheelbase>0.128</wheelbase>
-        <wheel_separation>0.310</wheel_separation>
-        <wheel_radius>0.035</wheel_radius>
-        <odom_publish_frequency>50</odom_publish_frequency>
-        <odom_topic>odom</odom_topic>
-        <frame_id>odom</frame_id>
-        <child_frame_id>base_footprint</child_frame_id>
+<robot name="robot" xmlns:xacro="http://ros.org/wiki/xacro">
+  <xacro:arg name="laser_visual" default="false"/>
+  <xacro:arg name="imu_visual"   default="false"/>
+  <!-- ROS 2 Control -->
+  <gazebo>
+    <plugin filename="libgazebo_ros2_control.so" name="gazebo_ros2_control">
+      <robot_param>robot_description</robot_param>
+      <robot_param_node>robot_state_publisher</robot_param_node>
+      <parameters>$(find robot_simulation)/config/robot_controllers.yaml</parameters>
     </plugin>
   </gazebo>
-    <gazebo reference="base_scan">
-        <sensor name="gpu_lidar" type="gpu_ray">
-            <topic>scan</topic>
-            <update_rate>10</update_rate>
-            <visualize>true</visualize>
-            <frame_id>base_scan</frame_id>
-            <ignition_frame_id>base_scan</ignition_frame_id>
-            <ray>
-                <scan>
-                    <horizontal>
-                        <samples>360</samples>
-                        <resolution>1</resolution>
-                        <min_angle>-3.14159</min_angle>
-                        <max_angle>3.14159</max_angle>
-                    </horizontal>
-                </scan>
-                <range>
-                    <min>0.12</min>
-                    <max>10.0</max>
-                    <resolution>0.01</resolution>
-                </range>
-                <noise>
-                    <type>gaussian</type>
-                    <mean>0.0</mean>
-                    <stddev>0.01</stddev>
-                </noise>
-            </ray>
-        </sensor>
-    </gazebo>
+  <gazebo reference="base_link">
+    <material>Gazebo/DarkGrey</material>
+  </gazebo>
+  <!-- IMU Sensor (ROS2) -->
+  <gazebo reference="imu_link">
+    <sensor name="imu_sensor" type="imu">
+      <always_on>true</always_on>
+      <update_rate>200</update_rate>
+      <visualize>$(arg imu_visual)</visualize>
+      <imu>
+        <angular_velocity>
+          <x>
+            <noise type="gaussian">
+              <mean>0.0</mean>
+              <stddev>2e-4</stddev>
+              <bias_mean>0.0000075</bias_mean>
+              <bias_stddev>0.0000008</bias_stddev>
+            </noise>
+          </x>
+          <y>
+            <noise type="gaussian">
+              <mean>0.0</mean>
+              <stddev>2e-4</stddev>
+              <bias_mean>0.0000075</bias_mean>
+              <bias_stddev>0.0000008</bias_stddev>
+            </noise>
+          </y>
+          <z>
+            <noise type="gaussian">
+              <mean>0.0</mean>
+              <stddev>2e-4</stddev>
+              <bias_mean>0.0000075</bias_mean>
+              <bias_stddev>0.0000008</bias_stddev>
+            </noise>
+          </z>
+        </angular_velocity>
+        <linear_acceleration>
+          <x>
+            <noise type="gaussian">
+              <mean>0.0</mean>
+              <stddev>1.7e-2</stddev>
+              <bias_mean>0.1</bias_mean>
+              <bias_stddev>0.001</bias_stddev>
+            </noise>
+          </x>
+          <y>
+            <noise type="gaussian">
+              <mean>0.0</mean>
+              <stddev>1.7e-2</stddev>
+              <bias_mean>0.1</bias_mean>
+              <bias_stddev>0.001</bias_stddev>
+            </noise>
+          </y>
+          <z>
+            <noise type="gaussian">
+              <mean>0.0</mean>
+              <stddev>1.7e-2</stddev>
+              <bias_mean>0.1</bias_mean>
+              <bias_stddev>0.001</bias_stddev>
+            </noise>
+          </z>
+        </linear_acceleration>
+      </imu>
+      <plugin name="imu_plugin" filename="libgazebo_ros_imu_sensor.so">
+        <ros>
+          <namespace>/</namespace>
+          <remapping>~/out:=imu</remapping>
+        </ros>
+        <initial_orientation_as_reference>false</initial_orientation_as_reference>
+      </plugin>
+    </sensor>
+    <material>Gazebo/FlatBlack</material>
+  </gazebo>
+  <!-- Laser Scanner (ROS2) -->
+  <gazebo reference="base_scan">
+    <material>Gazebo/FlatBlack</material>
+    <sensor name="lds_lfcd_sensor" type="gpu_ray">
+      <pose>0 0 0 0 0 0</pose>
+      <visualize>$(arg laser_visual)</visualize>
+      <update_rate>5</update_rate>
+      <ray>
+        <scan>
+          <horizontal>
+            <samples>360</samples>
+            <resolution>1</resolution>
+            <min_angle>0.0</min_angle>
+            <max_angle>6.28319</max_angle>
+          </horizontal>
+        </scan>
+        <range>
+          <min>0.120</min>
+          <max>3.5</max>
+          <resolution>0.015</resolution>
+        </range>
+        <noise>
+          <type>gaussian</type>
+          <mean>0.0</mean>
+          <stddev>0.01</stddev>
+        </noise>
+      </ray>
+      <plugin name="gazebo_ros_lds_lfcd_controller" filename="libgazebo_ros_ray_sensor.so">
+        <ros>
+          <namespace>/</namespace>
+          <remapping>~/out:=scan</remapping>
+        </ros>
+        <output_type>sensor_msgs/LaserScan</output_type>
+        <frame_name>base_scan</frame_name>
+      </plugin>
+    </sensor>
+  </gazebo>
 </robot>

File: robot_simulation/urdf/robot.urdf.xacro (robot description, xacro)
@@ -1,179 +1,90 @@
 <?xml version="1.0" ?>
-<robot name="turtlebot3_waffle_pi" xmlns:xacro="http://ros.org/wiki/xacro">
-  <!-- Init colour -->
-  <material name="black">
-      <color rgba="0.0 0.0 0.0 1.0"/>
-  </material>
-  <material name="dark">
-    <color rgba="0.3 0.3 0.3 1.0"/>
-  </material>
-  <material name="light_black">
-    <color rgba="0.4 0.4 0.4 1.0"/>
-  </material>
-  <material name="blue">
-    <color rgba="0.0 0.0 0.8 1.0"/>
-  </material>
-  <material name="green">
-    <color rgba="0.0 0.8 0.0 1.0"/>
-  </material>
-  <material name="grey">
-    <color rgba="0.5 0.5 0.5 1.0"/>
-  </material>
-  <material name="orange">
-    <color rgba="1.0 0.4235 0.0392 1.0"/>
-  </material>
-  <material name="brown">
-    <color rgba="0.8706 0.8118 0.7647 1.0"/>
-  </material>
-  <material name="red">
-    <color rgba="0.8 0.0 0.0 1.0"/>
-  </material>
-  <material name="white">
-    <color rgba="1.0 1.0 1.0 1.0"/>
-  </material>
+<robot name="robot" xmlns:xacro="http://ros.org/wiki/xacro">
+  <xacro:include filename="$(find robot_simulation)/urdf/common_properties.xacro"/>
+  <xacro:include filename="$(find robot_simulation)/urdf/robot.gazebo.xacro"/>
+  <xacro:include filename="$(find robot_simulation)/urdf/mecanum_description.urdf.xacro"/>
+  <xacro:include filename="$(find robot_simulation)/urdf/mecanum_description.gazebo.xacro"/>
+  <xacro:property name="PI" value="3.1415926535897931"/>
+  <xacro:property name="b_diam" value="0.13755" />    <!-- base diameter -->
+  <xacro:property name="b_height" value="0.14413" />  <!-- base height -->
   <link name="base_footprint"/>
   <joint name="base_joint" type="fixed">
     <parent link="base_footprint"/>
-    <child link="base_link" />
-    <origin xyz="0 0 0.010" rpy="0 0 0"/>
+    <child link="base_link"/>
+    <origin xyz="0.0 0.0 0.010" rpy="0 0 0"/>
   </joint>
   <link name="base_link">
     <visual>
-      <origin xyz="-0.064 0 0.0" rpy="0 0 0"/>
+      <origin xyz="0.0 0 0.0" rpy="0 0 0"/>
       <geometry>
-        <mesh filename="package://robot_simulation/models/robot/meshes/bases/waffle_pi_base.stl" scale="0.001 0.001 0.001"/>
+        <mesh filename="package://robot_simulation/models/robot/meshes/bases/burger_base_4_servos.stl" scale="0.001 0.001 0.001"/>
       </geometry>
       <material name="light_black"/>
     </visual>
     <collision>
-      <origin xyz="-0.064 0 0.047" rpy="0 0 0"/>
+      <origin xyz="0.0 0.0 ${b_height/2}" rpy="0 0 0"/>
       <geometry>
-        <box size="0.266 0.266 0.094"/>
+        <box size="0.140 0.140 0.143"/>
       </geometry>
     </collision>
     <inertial>
       <origin xyz="0 0 0" rpy="0 0 0"/>
-      <mass value="1.3729096e+00"/>
-      <inertia ixx="8.7002718e-03" ixy="-4.7576583e-05" ixz="1.1160499e-04"
-               iyy="8.6195418e-03" iyz="-3.5422299e-06"
-               izz="1.4612727e-02" />
+      <mass value="20.0"/>
+      <inertia ixx="1.0" ixy="0.0" ixz="0.0"
+               iyy="1.0" iyz="0.0"
+               izz="1.0" />
     </inertial>
   </link>
-  <joint name="wheel_front_left_joint" type="continuous">
-    <parent link="base_link"/>
-    <child link="wheel_front_left_link"/>
-    <origin xyz="0.0 0.155 0.023" rpy="0 0 0"/>
-    <axis xyz="0 1 0"/>
-  </joint>
-  <link name="wheel_front_left_link">
-    <visual>
-      <origin xyz="0 0 0" rpy="0 0 0"/>
-      <geometry>
-        <mesh filename="package://robot_simulation/models/robot/meshes/wheels/mecanum_wheel_left.stl" scale="0.0007 0.0007 0.0007"/>
-      </geometry>
-      <material name="dark"/>
-    </visual>
-    <collision>
-      <origin xyz="0 0 0" rpy="1.57 0 0"/>
-      <geometry>
-        <cylinder length="0.018" radius="0.035"/>
-      </geometry>
-    </collision>
-    <inertial>
-      <origin xyz="0 0 0" />
-      <mass value="2.8498940e-02" />
-      <inertia ixx="1.1175580e-05" ixy="-4.2369783e-11" ixz="-5.9381719e-09"
-               iyy="1.1192413e-05" iyz="-1.4400107e-11"
-               izz="2.0712558e-05" />
-      </inertial>
-  </link>
-  <joint name="wheel_rear_left_joint" type="continuous">
-    <parent link="base_link"/>
-    <child link="wheel_rear_left_link"/>
-    <origin xyz="-0.128 0.155 0.023" rpy="0 0 0"/>
-    <axis xyz="0 1 0"/>
-  </joint>
-  <link name="wheel_rear_left_link">
-    <visual>
-      <origin xyz="0 0 0" rpy="0 0 0"/>
-      <geometry>
-        <mesh filename="package://robot_simulation/models/robot/meshes/wheels/mecanum_wheel_right.stl" scale="0.0007 0.0007 0.0007"/>
-      </geometry>
-      <material name="dark"/>
-    </visual>
-    <collision>
-      <origin xyz="0 0 0" rpy="1.57 0 0"/>
-      <geometry>
-        <cylinder length="0.018" radius="0.035"/>
-      </geometry>
-    </collision>
-    <inertial>
-      <origin xyz="0 0 0" />
-      <mass value="2.8498940e-02" />
-      <inertia ixx="1.1175580e-05" ixy="-4.2369783e-11" ixz="-5.9381719e-09"
-               iyy="1.1192413e-05" iyz="-1.4400107e-11"
-               izz="2.0712558e-05" />
-      </inertial>
-  </link>
-  <joint name="wheel_front_right_joint" type="continuous">
-    <parent link="base_link"/>
-    <child link="wheel_front_right_link"/>
-    <origin xyz="0.0 -0.155 0.023" rpy="0 0 0"/>
-    <axis xyz="0 1 0"/>
-  </joint>
-  <link name="wheel_front_right_link">
-    <visual>
-      <origin xyz="0 0 0" rpy="0 0 0"/>
-      <geometry>
-        <mesh filename="package://robot_simulation/models/robot/meshes/wheels/mecanum_wheel_right.stl" scale="0.0007 0.0007 0.0007"/>
-      </geometry>
-      <material name="dark"/>
-    </visual>
-    <collision>
-      <origin xyz="0 0 0" rpy="1.57 0 0"/>
-      <geometry>
-        <cylinder length="0.018" radius="0.035"/>
-      </geometry>
-    </collision>
-    <inertial>
-      <origin xyz="0 0 0" />
-      <mass value="2.8498940e-02" />
-      <inertia ixx="1.1175580e-05" ixy="-4.2369783e-11" ixz="-5.9381719e-09"
-               iyy="1.1192413e-05" iyz="-1.4400107e-11"
-               izz="2.0712558e-05" />
-      </inertial>
-  </link>
-  <joint name="wheel_rear_right_joint" type="continuous">
-    <parent link="base_link"/>
-    <child link="wheel_rear_right_link"/>
-    <origin xyz="-0.128 -0.155 0.023" rpy="0 0 0"/>
-    <axis xyz="0 1 0"/>
-  </joint>
-  <link name="wheel_rear_right_link">
-    <visual>
-      <origin xyz="0 0 0" rpy="0 0 0"/>
-      <geometry>
-        <mesh filename="package://robot_simulation/models/robot/meshes/wheels/mecanum_wheel_left.stl" scale="0.0007 0.0007 0.0007"/>
-      </geometry>
-      <material name="dark"/>
-    </visual>
-    <collision>
-      <origin xyz="0 0 0" rpy="1.57 0 0"/>
-      <geometry>
-        <cylinder length="0.018" radius="0.035"/>
-      </geometry>
-    </collision>
-    <inertial>
-      <origin xyz="0 0 0" />
-      <mass value="2.8498940e-02" />
-      <inertia ixx="1.1175580e-05" ixy="-4.2369783e-11" ixz="-5.9381719e-09"
-               iyy="1.1192413e-05" iyz="-1.4400107e-11"
-               izz="2.0712558e-05" />
-      </inertial>
-  </link>
+  <xacro:mecanum_wheel1 base_name="base_link" base_diam="b_diam" suffix="rf" right="1"   front="1"/>
+  <xacro:mecanum_wheel2 base_name="base_link" base_diam="b_diam" suffix="lf" right="-1"   front="1"/>
+  <xacro:mecanum_wheel2 base_name="base_link" base_diam="b_diam" suffix="rb" right="1"   front="-1"/>
+  <xacro:mecanum_wheel1 base_name="base_link" base_diam="b_diam" suffix="lb" right="-1"   front="-1"/>
+  <!-- ROS 2 Control -->
+  <ros2_control name="GazeboSystem" type="system">
+    <hardware>
+      <plugin>gazebo_ros2_control/GazeboSystem</plugin>
+    </hardware>
+    <!-- Right Front Wheel -->
+    <joint name="mecanum_rf_joint">
+      <command_interface name="velocity">
+        <param name="min">-10</param>
+        <param name="max">10</param>
+      </command_interface>
+      <state_interface name="position"/>
+      <state_interface name="velocity"/>
+    </joint>
+    <!-- Left Front Wheel -->
+    <joint name="mecanum_lf_joint">
+      <command_interface name="velocity">
+        <param name="min">-10</param>
+        <param name="max">10</param>
+      </command_interface>
+      <state_interface name="position"/>
+      <state_interface name="velocity"/>
+    </joint>
+    <!-- Right Back Wheel -->
+    <joint name="mecanum_rb_joint">
+      <command_interface name="velocity">
+        <param name="min">-10</param>
+        <param name="max">10</param>
+      </command_interface>
+      <state_interface name="position"/>
+      <state_interface name="velocity"/>
+    </joint>
+    <!-- Left Back Wheel -->
+    <joint name="mecanum_lb_joint">
+      <command_interface name="velocity">
+        <param name="min">-10</param>
+        <param name="max">10</param>
+      </command_interface>
+      <state_interface name="position"/>
+      <state_interface name="velocity"/>
+    </joint>
+  </ros2_control>
+  <!-- Sensors block -->
   <joint name="imu_joint" type="fixed">
     <parent link="base_link"/>
     <child link="imu_link"/>
-    <origin xyz="0.0 0 0.068" rpy="0 0 0"/>
+    <origin xyz="-0.032 0 0.068" rpy="0 0 0"/>
   </joint>
   <link name="imu_link"/>
@@ -181,5 +92,5 @@
     <parent link="base_link"/>
     <child link="base_scan"/>
-    <origin xyz="-0.064 0 0.122" rpy="0 0 0"/>
+    <origin xyz="-0.032 0 0.172" rpy="0 0 0"/>
   </joint>
   <link name="base_scan">
@@ -205,29 +116,3 @@
     </inertial>
   </link>
-  <joint name="camera_joint" type="fixed">
-    <origin xyz="0.073 -0.011 0.084" rpy="0 0 0"/>
-    <parent link="base_link"/>
-    <child link="camera_link"/>
-  </joint>
-  <link name="camera_link">
-    <collision>
-      <origin xyz="0.005 0.011 0.013" rpy="0 0 0"/>
-      <geometry>
-        <box size="0.015 0.030 0.027"/>
-      </geometry>
-    </collision>
-  </link>
-  <joint name="camera_rgb_joint" type="fixed">
-    <origin xyz="0.003 0.011 0.009" rpy="0 0 0"/>
-    <parent link="camera_link"/>
-    <child link="camera_rgb_frame"/>
-  </joint>
-  <link name="camera_rgb_frame"/>
-  <joint name="camera_rgb_optical_joint" type="fixed">
-    <origin xyz="0 0 0" rpy="-1.57 0 -1.57"/>
-    <parent link="camera_rgb_frame"/>
-    <child link="camera_rgb_optical_frame"/>
-  </joint>
-  <link name="camera_rgb_optical_frame"/>
-  <xacro:include filename="robot.gazebo.xacro" />
 </robot>
